File: Audio Interface/Audio Interface.kicad_pcb (KiCad board)
At the start: 2 copper layers, 36 parts, among them J1 USB_C_Receptacle_USB2.0_16P, J2 NRJ4HH-1, J3 NRJ4HH-1, SW1 SW_Push, SW2 SW_Push, SW3 SW_Push, U1 PCM2903, U2 USBLC6-2SC6, U3 AMS1117-3.3, Y1 12MHz

Commit message: commit 2 of kicad files test
Parts:
- moved J3 38.3 mm to (170.7, 102.4)
- moved J2 38.3 mm to (170.3, 68.7)
- moved C7 31.8 mm to (155.8, 136.1)
- moved R18 31.8 mm to (163.7, 136.1)
- moved SW3 31.8 mm to (170.8, 135.7)
- moved C6 28.9 mm to (156.2, 127.9)
- moved R17 28.9 mm to (164.0, 128.6)
- moved SW2 28.9 mm to (170.8, 129.1)
- moved R16 25.8 mm to (163.8, 122.5)
- moved SW1 25.8 mm to (170.6, 122.5)
- moved C5 25.8 mm to (157.5, 122.5)
- moved R4 23.8 mm to (164.6, 57.0)
- moved D1 23.8 mm to (176.3, 57.0)
- moved C11 19.7 mm to (125.2, 110.3)
- moved C12 19.7 mm to (111.6, 109.8)
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Other:
- board text added: "Mechanical - USB must line up with back panel - Mounting hole placement!! - front buttons will be flywire not pcb mounted"

Commit message: ordered board
Parts:
- removed J2: NRJ4HH-1, Connector_Audio:Jack_6.35mm_Neutrik_NRJ4HH-1_Horizontal
- removed R2: 1k5, Resistor_SMD:R_0402_1005Metric_Pad0.72x0.64mm_HandSolder
- added C10: 100nF, Capacitor_SMD:C_0402_1005Metric_Pad0.74x0.62mm_HandSolder, F.Cu at (106.6, 69.8)
- added C13: 100nF, Capacitor_SMD:C_0402_1005Metric_Pad0.74x0.62mm_HandSolder, F.Cu at (93.7, 71.6)
- added C14: 100nF, Capacitor_SMD:C_0402_1005Metric_Pad0.74x0.62mm_HandSolder, F.Cu at (94.7, 70.4)
- added C15: 100nF, Capacitor_SMD:C_0402_1005Metric_Pad0.74x0.62mm_HandSolder, F.Cu at (94.4, 75.3)
- added C18: 100nF, Capacitor_SMD:C_0402_1005Metric_Pad0.74x0.62mm_HandSolder, F.Cu at (94.4, 76.5)
- added J4: NRJ4HH-1, Connector_Audio:Jack_6.35mm_Neutrik_NRJ4HH-1_Horizontal, F.Cu at (104.3, 49.5)
- added TP5: TestPoint, TestPoint:TestPoint_Pad_D1.0mm, F.Cu at (81.8, 74.7)
- J3: footprint Connector_Audio:Jack_6.35mm_Neutrik_NRJ4HH-1_Horizontal -> Connector_PinHeader_2.54mm:PinHeader_1x04_P2.54mm_Vertical
- Y1: footprint Crystal:Crystal_SMD_HC49-SD_HandSoldering -> Crystal:Crystal_SMD_3225-4Pin_3.2x2.5mm_HandSoldering
- moved J3 105.6 mm to (79.4, 49.5), turned to 90 degrees
- moved C1 87.2 mm to (79.5, 68.5), turned to 180 degrees
- moved SW2 84.8 mm to (115.0, 65.2)
- moved SW3 84.2 mm to (115.0, 72.7)
- moved C3 83.8 mm to (79.5, 67.0), turned to 180 degrees
- moved C4 82.3 mm to (79.5, 65.7), turned to 180 degrees
- moved C2 82.2 mm to (82.4, 70.3)
- moved R17 82.2 mm to (111.7, 65.2), turned to 180 degrees
- moved R18 81.9 mm to (111.8, 72.7), turned to 180 degrees
- moved SW1 77.3 mm to (115.1, 68.7)
- moved R16 74.7 mm to (111.9, 68.7), turned to 180 degrees
- moved U3 74.5 mm to (83.7, 67.0)
- moved C7 73.1 mm to (116.4, 74.6)
- moved C6 72.8 mm to (116.3, 67.0)
- moved TP1 68.3 mm to (81.8, 72.0), turned to 90 degrees
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Connections:
- net /USB_D+_IN renamed /USB_IN+
- net /USB_D+_OUT renamed /USB_OUT+
- net /USB_D-_IN renamed /USB_IN-
- net /USB_D-_OUT renamed /USB_OUT-
Routing:
- net +3V3: track 0.00 -> 90.2 mm, vias 0 -> 2
- net /VBUS: track 0.00 -> 60.6 mm, vias 0 -> 5
- net Net-(U1-VINL): track 0.00 -> 29.5 mm
- net Net-(U1-VOUTL): track 0.00 -> 25.1 mm
- net /Guitar_IN: track 0.00 -> 23.7 mm
- net GND: track 0.00 -> 23.1 mm, vias 0 -> 29
- net /Volume Down: track 0.00 -> 19.1 mm
- net /Volume Up: track 0.00 -> 16.1 mm
- net /Mute: track 0.00 -> 15.6 mm
- net /USB_OUT-: track 0.00 -> 13.7 mm
- net /USB_OUT+: track 0.00 -> 13.6 mm
- net Net-(U1-XTO): track 0.00 -> 13.1 mm
- net /USB_IN-: track 0.00 -> 10.9 mm
- net /USB_IN+: track 0.00 -> 10.2 mm
- net Net-(U1-XTI): track 0.00 -> 7.41 mm
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- added copper zone on B.Cu, net GND
- added copper zone on F.Cu, net GND
Other:
- board outline added: 45.4 x 40.9 mm
- board text added: "3V3"
- board text added: "5V"
- board text added: "AUX"
- board text added: "Audio Interface V1"
- board text added: "GND"
- board text added: "Guitar"
- board text added: "Xander Beal 8/1/24 11:57PM"
