File: Audio Interface/Audio Interface.kicad_sch (KiCad schematic)
At the start: 36 parts, among them J1 USB_C_Receptacle_USB2.0_16P, J2 NRJ4HH-1, J3 NRJ4HH-1, SW1 SW_Push, SW2 SW_Push, SW3 SW_Push, U1 PCM2903, U2 USBLC6-2SC6, U3 AMS1117-3.3, Y1 12MHz

Commit message: ordered board
Parts:
- removed J2: NRJ4HH-1, Connector_Audio:Jack_6.35mm_Neutrik_NRJ4HH-1_Horizontal, symbol Connector_Audio:NRJ4HH-1
- removed R2: 1k5, Resistor_SMD:R_0402_1005Metric_Pad0.72x0.64mm_HandSolder, symbol Device:R
- added C10, C13, C14, C15, C18: 100nF, Capacitor_SMD:C_0402_1005Metric_Pad0.74x0.62mm_HandSolder, symbol Device:C
- added J4: NRJ4HH-1, Connector_Audio:Jack_6.35mm_Neutrik_NRJ4HH-1_Horizontal, symbol Connector_Audio:NRJ4HH-1
- added TP5: TestPoint, TestPoint:TestPoint_Pad_D1.0mm, symbol Connector:TestPoint
- J3: footprint Connector_Audio:Jack_6.35mm_Neutrik_NRJ4HH-1_Horizontal -> Connector_PinHeader_2.54mm:PinHeader_1x04_P2.54mm_Vertical
- Y1: footprint Crystal:Crystal_SMD_HC49-SD_HandSoldering -> Crystal:Crystal_SMD_3225-4Pin_3.2x2.5mm_HandSoldering
Connections:
- net +3V3: now also C10.1, C13.1, C14.1, C15.1, C18.1
- net AUX_OUT: now also J3.2, J3.3; no longer J3.T, J3.TN
- net GND: now also J3.1, J3.4, C10.2, C13.2, C14.2, C15.2, C18.2, J4.G, J4.S, TP5.1; no longer J3.G, J3.S
- net Guitar_IN: now also J4.T, J4.TN
- net USB_D+_IN renamed USB_IN+
- net USB_D+_OUT renamed USB_OUT+
- net USB_D-_IN renamed USB_IN-
- net USB_D-_OUT renamed USB_OUT-
Other:
- moved on the sheet: C9
